Commit message: av1 files

File: src/my_robot_AV1/urdf/robot.urdf.xacro (robot description, xacro)
@@ -2,4 +2,3 @@
 <robot xmlns:xacro="http://www.ros.org/wiki/xacro" name="my_robot">
     <xacro:include filename="robot_core.xacro" />
-    <xacro:include filename="gazebo_control.xacro" />
 </robot>

File: src/my_robot_AV1/urdf/robot_core.xacro (robot description, xacro)
@@ -2,8 +2,15 @@
 <robot xmlns:xacro="http://www.ros.org/wiki/xacro" >
     <xacro:include filename="inertial_macros.xacro"/>
-    <material name="white"><color rgba="1 1 1 1" /></material>
-    <material name="blue"><color rgba="0.2 0.2 1 1" /></material>
-    <material name="black"><color rgba="0 0 0 1" /></material>
-    <link name="base_link"></link>
+    <material name="white">
+        <color rgba="1 1 1 1" />
+    </material>
+    <material name="blue">
+        <color rgba="0.2 0.2 1 1" />
+    </material>
+    <material name="black">
+        <color rgba="0 0 0 1" />
+    </material>
+    <link name="base_link">
+    </link>
     <joint name="chassis_joint" type="fixed">
         <parent link="base_link"/>
@@ -14,10 +21,14 @@
         <visual>
             <origin xyz="0.3 0 0.1"/>
-            <geometry><box size="0.6 0.4 0.2"/></geometry>
+            <geometry>
+                <box size="0.6 0.4 0.2"/>
+            </geometry>
             <material name="white"/>
         </visual>
         <collision>
             <origin xyz="0.3 0 0.1"/>
-            <geometry><box size="0.6 0.4 0.2"/></geometry>
+            <geometry>
+                <box size="0.6 0.4 0.2"/>
+            </geometry>
         </collision>
         <xacro:inertial_box mass="5.0" x="0.6" y="0.4" z="0.2">
@@ -25,4 +36,7 @@
         </xacro:inertial_box>
     </link>
+    <gazebo reference="chassis">
+        <material>Gazebo/White</material>
+    </gazebo>
     <joint name="left_wheel_joint" type="continuous">
         <parent link="base_link"/>
@@ -33,9 +47,13 @@
     <link name="left_wheel">
         <visual>
-            <geometry><cylinder radius="0.1" length="0.05"/></geometry>
+            <geometry>
+                <cylinder radius="0.1" length="0.05"/>
+            </geometry>
             <material name="blue"/>
         </visual>
         <collision>
-            <geometry><cylinder radius="0.1" length="0.05"/></geometry>
+            <geometry>
+                <cylinder radius="0.1" length="0.05"/>
+            </geometry>
         </collision>
         <xacro:inertial_cylinder mass="1.0" length="0.05" radius="0.1">
@@ -43,4 +61,7 @@
         </xacro:inertial_cylinder>
     </link>
+    <gazebo reference="left_wheel">
+        <material>Gazebo/Blue</material>
+    </gazebo>
     <joint name="right_wheel_joint" type="continuous">
         <parent link="base_link"/>
@@ -51,9 +72,13 @@
     <link name="right_wheel">
         <visual>
-            <geometry><cylinder radius="0.1" length="0.05"/></geometry>
+            <geometry>
+                <cylinder radius="0.1" length="0.05"/>
+            </geometry>
             <material name="blue"/>
         </visual>
         <collision>
-            <geometry><cylinder radius="0.1" length="0.05"/></geometry>
+            <geometry>
+                <cylinder radius="0.1" length="0.05"/>
+            </geometry>
         </collision>
         <xacro:inertial_cylinder mass="1.0" length="0.05" radius="0.1">
@@ -61,4 +86,7 @@
         </xacro:inertial_cylinder>
     </link>
+    <gazebo reference="right_wheel">
+        <material>Gazebo/Blue</material>
+    </gazebo>
     <joint name="caster_wheel_joint" type="fixed">
         <parent link="chassis"/>
@@ -68,9 +96,13 @@
     <link name="caster_wheel">
         <visual>
-            <geometry><sphere radius="0.1"/></geometry>
+            <geometry>
+                <sphere radius="0.1"/>
+            </geometry>
             <material name="black"/>
         </visual>
         <collision>
-            <geometry><sphere radius="0.1"/></geometry>
+            <geometry>
+                <sphere radius="0.1"/>
+            </geometry>
         </collision>
         <xacro:inertial_sphere mass="0.5" radius="0.1">
