Commit message: fix wheels

File: ros_ws/src/my_robot_description/urdf/mobile_base.xacro (robot description, xacro)
@@ -18,4 +18,11 @@
             <material name="blue" />
         </visual>
+        <collision>
+            <geometry>
+                <box size="${base_length} ${base_width} ${base_height}" />
+            </geometry>
+            <origin xyz="0 0 ${base_height / 2.0}" rpy="0 0 0" />
+        </collision>
+        <xacro:box_inertia m="5.0" l="${base_length}" w="${base_width}" h="${base_height}" xyz="0 0 ${base_height / 2.0}" rpy="0 0 0" />
     </link>
     <link name="left_wheel">
@@ -27,4 +34,11 @@
             <material name="red" />
         </visual>
+        <collision>
+            <geometry>
+                <cylinder radius="${wheel_radius}" length="${wheel_length}" />
+            </geometry>
+            <origin xyz="0 0 0" rpy="${pi / 2.0} 0 0" />
+        </collision>
+        <xacro:cylinder_inertia m="1.0" r="${wheel_radius}" h="${wheel_length}" xyz="0 0 0" rpy="${pi / 2.0} 0 0" />
     </link>
     <link name="right_wheel">
@@ -36,4 +50,11 @@
             <material name="red" />
         </visual>
+        <collision>
+            <geometry>
+                <cylinder radius="${wheel_radius}" length="${wheel_length}" />
+            </geometry>
+            <origin xyz="0 0 0" rpy="${pi / 2.0} 0 0" />
+        </collision>
+        <xacro:cylinder_inertia m="1.0" r="${wheel_radius}" h="${wheel_length}" xyz="0 0 0" rpy="${pi / 2.0} 0 0" />
     </link>
     <link name="caster_wheel">
@@ -45,4 +66,11 @@
             <material name="white" />
         </visual>
+        <collision>
+            <geometry>
+                <sphere radius="${wheel_radius / 2.0}" />
+            </geometry>
+            <origin xyz="0 0 0" rpy="0 0 0" />
+        </collision>
+        <xacro:sphere_inertia m="0.5" r="${wheel_radius / 2.0}" xyz="0 0 0" rpy="0 0 0" />
     </link>
     <joint name="base_joint" type="fixed">
@@ -68,12 +96,3 @@
         <origin xyz="${base_length / 3.0} 0 ${-wheel_radius / 2.0}" rpy="0 0 0" />
     </joint>
-    <collision>
-        <geometry>
-            <box size="${base_length} ${base_width} ${base_height}" />
-        </geometry>
-        <origin xyz="0 0 ${base_height / 2.0}" rpy="0 0 0" />
-    </collision>
-    <xacro:box_inertia m="5.0" l="${2*base_length}" w="${2*base_width}" h="${2*base_height}" xyz="0 0 ${base_height / 2.0}" rpy="0 0 0" />
-    <xacro:box_inertia m="5.0" l="${2*base_length}" w="${2*base_width}" h="${2*base_height}" xyz="0 0 ${base_height / 2.0}" rpy="0 0 0" />
-    <xacro:sphere_inertia m="0.5" r="${2*wheel_radius / 2.0}" xyz="0 0 0" rpy="0 0 0" />
 </robot>

File: ros_ws/src/my_robot_description/urdf/mobile_base_gazebo.xacro (robot description, xacro)
@@ -4,11 +4,11 @@
 	    <material>Gazebo/Blue</material>
     </gazebo>
-    <gazebo reference="right_wheel_link">
+    <gazebo reference="right_wheel">
         <material>Gazebo/Grey</material>
     </gazebo>
-    <gazebo reference="left_wheel_link">
+    <gazebo reference="left_wheel">
         <material>Gazebo/Grey</material>
     </gazebo>
-    <gazebo reference="caster_wheel_link">
+    <gazebo reference="caster_wheel">
         <material>Gazebo/Grey</material>
         <mu1 value="0.1" />
